Commit message: benchmarking

File: data/urdfs/mia_hand_on_ur10.urdf (robot description, URDF)
Before this commit: robot mia_hand_on_ur10, 25 links, 24 joints
Links:
- link ur10_base_link_inertia: geometry collision cylinder length=0.038 radius=0.07498; visual mesh filename=../meshes/dae/shape0.001.dae scale=1.0 1.0 1.0
- link ur10_forearm_link: geometry collision cylinder length=0.67816 radius=0.0601; visual mesh filename=../meshes/dae/shape4.dae scale=1.0 1.0 1.0
- link ur10_shoulder_link: geometry collision cylinder length=0.17711 radius=0.07548; visual mesh filename=../meshes/dae/shape2.001.dae scale=1.0 1.0 1.0
- link ur10_upper_arm_link: geometry collision cylinder length=0.74884 radius=0.07534; visual mesh filename=../meshes/dae/shape3.001.dae scale=1.0 1.0 1.0
- link ur10_wrist_1_link: geometry collision cylinder length=0.11882 radius=0.04551; visual mesh filename=../meshes/dae/shape2.003.dae scale=1.0 1.0 1.0
- link ur10_wrist_2_link: geometry collision cylinder length=0.10009 radius=0.04563; visual mesh filename=../meshes/dae/shape2.004.dae scale=1.0 1.0 1.0
- link ur10_wrist_3_link: geometry collision cylinder length=0.09007 radius=0.04497; visual mesh filename=../meshes/dae/shape0.006.dae scale=1.0 1.0 1.0

Commit message: benchmarking

File: data/urdfs/mia_hand_on_ur10.urdf (robot description, URDF)
Before this commit: robot mia_hand_on_ur10, 25 links, 24 joints
Links:
- link arm_base: mass 0.82574 -> None; geometry collision box size=0.20000 0.20000 1.00000
- link flange: geometry 
- link hand_ee_link: mass 1e-05 -> None
- link index_fle: mass 0.01113 -> None
- link index_sensor: mass 0.01765 -> None; geometry collision cylinder length=0.01426 radius=0.00713; collision cylinder length=0.03037 radius=0.00796
- link little_fle: mass 0.0207 -> None; geometry collision cylinder length=0.02993 radius=0.00760; collision cylinder length=0.03044 radius=0.00783
- link middle_fle: mass 0.0121 -> None
- link middle_sensor: mass 0.0177 -> None; geometry collision cylinder length=0.01183 radius=0.00683; collision cylinder length=0.03824 radius=0.00813
- link palm: mass 0.274 -> None; geometry collision box size=0.06241 0.05638 0.02858; collision box size=0.07264 0.04753 0.03326
- link ring_fle: mass 0.0263 -> None; geometry collision cylinder length=0.02993 radius=0.00760; collision cylinder length=0.03683 radius=0.00783
- link thumb_fle: mass 0.0592 -> None; geometry collision cylinder length=0.05502 radius=0.01169; collision cylinder length=0.05982 radius=0.01271
- link thumb_opp: mass 0.013 -> None; geometry 
- link thumb_sensor: mass 0.00064 -> None
- link ur10_base_link_inertia: mass 4.0 -> None; geometry collision box size=0.14996 0.16710 0.03800; visual mesh filename=../meshes/stl/base.stl scale=1.00000 1.00000 1.00000
- link ur10_forearm_link: mass 3.87 -> None; geometry collision box size=0.12020 0.13634 0.67816; visual mesh filename=../meshes/stl/forearm.stl scale=1.00000 1.00000 1.00000
- link ur10_shoulder_link: mass 7.778 -> None; geometry collision box size=0.15095 0.16137 0.17711; visual mesh filename=../meshes/stl/shoulder.stl scale=1.00000 1.00000 1.00000
- link ur10_upper_arm_link: mass 12.93 -> None; geometry collision box size=0.15068 0.17726 0.74884; collision box size=0.15068 0.17726 0.74884
- link ur10_wrist_1_link: mass 1.96 -> None; geometry collision box size=0.09102 0.10007 0.11882; visual mesh filename=../meshes/stl/wrist1.stl scale=1.00000 1.00000 1.00000
- link ur10_wrist_2_link: mass 1.96 -> None; geometry collision box size=0.09126 0.11887 0.10009; visual mesh filename=../meshes/stl/wrist2.stl scale=1.00000 1.00000 1.00000
- link ur10_wrist_3_link: mass 0.202 -> None; geometry collision box size=0.08993 0.03050 0.09007; visual mesh filename=../meshes/stl/wrist3.stl scale=1.00000 1.00000 1.00000
Joints:
- joint arm_base_to_arm: origin xyz=0 0 1.0 rpy=0 0 0 -> xyz=0.00000 0.00000 1.00000 rpy=0.00000 0.00000 0.00000
- joint j_index_fle: axis 0 0 1.0 -> -0.00000 0.00000 1.00000; limit lower=-1.4 upper=1.4 effort=1.75 velocity=3.14 -> lower=-1.40000 upper=1.40000 effort=1.75000 velocity=3.14000
- joint j_index_sensor: origin xyz=-0.0004 0.02424 -0.00018 rpy=0.00063 -0.00021 0.17208 -> xyz=-0.00040 0.02424 -0.00018 rpy=0.00063 -0.00021 0.17208
- joint j_little_fle: axis 0 0 1.0 -> -0.00000 0.00000 1.00000; limit lower=0 upper=1.39626 effort=1.75 velocity=3.14 -> lower=0 upper=1.39626 effort=1.75000 velocity=3.14000; origin xyz=-0.02786 0.10733 -0.02061 rpy=1.27834 1.77592 1.62718 -> xyz=-0.02786 0.10733 -0.02061 rpy=-1.86325 1.36567 -1.51441
- joint j_middle_sensor: origin xyz=0.00044 0.0255 0 rpy=0 0 0 -> xyz=0.00044 0.02550 0.00000 rpy=0.00000 0.00000 -0.00000
- joint j_mrl_fle: axis 0 0 1.0 -> -0.00000 0.00000 1.00000; limit lower=0 upper=1.39626 effort=1.75 velocity=3.14 -> lower=0 upper=1.39626 effort=1.75000 velocity=3.14000
- joint j_ring_fle: axis 0 0 1.0 -> -0.00000 0.00000 1.00000; limit lower=0 upper=1.39626 effort=1.75 velocity=3.14 -> lower=0 upper=1.39626 effort=1.75000 velocity=3.14000; origin xyz=-0.01225 0.11203 -0.02394 rpy=1.15081 1.68124 1.32178 -> xyz=-0.01225 0.11203 -0.02394 rpy=-1.99078 1.46035 -1.81981
- joint j_thumb_fle: axis 0 0 1.0 -> -0.00000 0.00000 1.00000; limit lower=0 upper=1.1345 effort=3.5 velocity=1.57 -> lower=0 upper=1.13450 effort=3.50000 velocity=1.57000; origin xyz=-3e-05 -1e-05 -0.00899 rpy=-1.57091 0.43822 1.57067 -> xyz=-0.00003 -0.00001 -0.00899 rpy=-1.57091 0.43822 1.57066
- joint j_thumb_opp: axis 0 0 1.0 -> -0.00000 0.00000 1.00000; limit lower=-0.628 upper=0 effort=3.5 velocity=4.0 -> lower=-0.62800 upper=0.00000 effort=3.50000 velocity=4.00000
- joint j_thumb_sensor: origin xyz=0 0.009 0 rpy=1.5708 0 0 -> xyz=-0.00001 0.00900 0.00000 rpy=1.57080 0.00000 -0.00000
- joint palm_to_flange: origin xyz=0 0 0 rpy=0 0 0 -> xyz=0.00000 0.00000 -0.00000 rpy=0.00000 0.00000 0.00000
- joint palm_to_hand_ee_link: origin xyz=0 0.13 0.03 rpy=-0.65 0 0 -> xyz=0.00000 0.13000 0.03000 rpy=-0.65000 -0.00000 -0.00000
- joint ur10_base_link-base_fixed_joint: origin xyz=0 0 0 rpy=0 0 -3.14159 -> xyz=0.00000 0.00000 0.00000 rpy=0.00000 0.00000 -3.14159
- joint ur10_base_link-base_link_inertia: origin xyz=0 0 0 rpy=0 0 -3.14159 -> xyz=0.00000 0.00000 0.00000 rpy=0.00000 0.00000 -3.14159
- joint ur10_elbow_joint: axis 0 0 1.0 -> 0.00000 0.00000 1.00000; limit lower=-3.14159 upper=3.14159 effort=150.0 velocity=3.14159 -> lower=-3.14159 upper=3.14159 effort=150.00000 velocity=3.14159; origin xyz=-0.612 0 0 rpy=0 0 0 -> xyz=-0.61200 0.00000 0.00000 rpy=-0.00000 0.00000 0.00000
- joint ur10_flange-tool0: origin xyz=0 0 0 rpy=1.5708 0 1.5708 -> xyz=0.00000 0.00000 0.00000 rpy=1.57080 -0.00000 1.57080
- joint ur10_shoulder_lift_joint: axis 0 0 1.0 -> 0.00000 0.00000 1.00000; limit lower=-6.28319 upper=6.28319 effort=330.0 velocity=2.0944 -> lower=-6.28319 upper=6.28319 effort=330.00000 velocity=2.09440; origin xyz=0 0 0 rpy=1.5708 0 0 -> xyz=0.00000 0.00000 0.00000 rpy=1.57080 0.00000 0.00000
- joint ur10_shoulder_pan_joint: axis 0 0 1.0 -> 0.00000 0.00000 1.00000; limit lower=-6.28319 upper=6.28319 effort=330.0 velocity=2.0944 -> lower=-6.28319 upper=6.28319 effort=330.00000 velocity=2.09440; origin xyz=0 0 0.1273 rpy=0 0 0 -> xyz=0.00000 0.00000 0.12730 rpy=0.00000 0.00000 0.00000
- joint ur10_to_mia: origin xyz=0 0 0.022 rpy=1.57079 0 -1.5708 -> xyz=-0.00000 -0.00000 0.02200 rpy=1.57079 0.00000 -1.57080
- joint ur10_wrist_1_joint: axis 0 0 1.0 -> 0.00000 0.00000 1.00000; limit lower=-6.28319 upper=6.28319 effort=56.0 velocity=3.14159 -> lower=-6.28319 upper=6.28319 effort=56.00000 velocity=3.14159; origin xyz=-0.5723 0 0.16394 rpy=0 0 0 -> xyz=-0.57230 -0.00000 0.16394 rpy=-0.00000 0.00000 0.00000
- joint ur10_wrist_2_joint: axis 0 0 1.0 -> 0.00000 0.00000 1.00000; limit lower=-6.28319 upper=6.28319 effort=56.0 velocity=3.14159 -> lower=-6.28319 upper=6.28319 effort=56.00000 velocity=3.14159; origin xyz=0 -0.1157 0 rpy=1.5708 0 0 -> xyz=-0.00000 -0.11570 0.00000 rpy=1.57080 0.00000 -0.00000
- joint ur10_wrist_3-flange: origin xyz=0 0 0 rpy=-1.5708 -1.5708 0 -> xyz=0.00000 0.00000 0.00000 rpy=1.57080 -1.57080 -3.14159
- joint ur10_wrist_3_joint: axis 0 0 1.0 -> 0.00000 0.00000 1.00000; limit lower=-6.28319 upper=6.28319 effort=56.0 velocity=3.14159 -> lower=-6.28319 upper=6.28319 effort=56.00000 velocity=3.14159; origin xyz=0 0.0922 0 rpy=-1.5708 0 0 -> xyz=-0.00000 0.09220 0.00000 rpy=-1.57080 0.00000 -0.00000
- joint world_to_robot: origin xyz=0 0 0 rpy=0 0 0 -> xyz=0.00000 0.00000 0.00000 rpy=0.00000 0.00000 0.00000
