Commit message: benchmarking

File: data/urdfs/nao.urdf (robot description, URDF)
Before this commit: robot NaoH25V40, 83 links, 82 joints
Links:
- link Head: geometry collision box size=0.11936 0.13267 0.11439; visual mesh filename=../meshes/stl/HeadPitch_0.10.stl scale=0.10000 0.10000 0.10000
- link LAnklePitch: geometry collision box size=0.07146 0.03136 0.06369; visual mesh filename=../meshes/stl/LAnklePitch_0.10.stl scale=0.10000 0.10000 0.10000
- link LBicep: geometry collision box size=0.16906 0.06238 0.08158; visual mesh filename=../meshes/stl/LShoulderRoll_0.10.stl scale=0.10000 0.10000 0.10000
- link LFinger11_link: mass 1e-05 -> 0.00000; geometry collision box size=0.01954 0.01519 0.01232; visual mesh filename=../meshes/stl/LFinger11_0.10.stl scale=0.10000 0.10000 0.10000
- link LFinger12_link: mass 1e-05 -> 0.00000; geometry collision box size=0.01954 0.01519 0.01232; visual mesh filename=../meshes/stl/LFinger12_0.10.stl scale=0.10000 0.10000 0.10000
- link LFinger13_link: mass 1e-05 -> 0.00000; geometry collision box size=0.01973 0.01591 0.01120; visual mesh filename=../meshes/stl/LFinger13_0.10.stl scale=0.10000 0.10000 0.10000
- link LFinger21_link: mass 1e-05 -> 0.00000; geometry collision box size=0.01954 0.01599 0.01211; visual mesh filename=../meshes/stl/LFinger21_0.10.stl scale=0.10000 0.10000 0.10000
- link LFinger22_link: mass 1e-05 -> 0.00000; geometry collision box size=0.01954 0.01599 0.01211; visual mesh filename=../meshes/stl/LFinger22_0.10.stl scale=0.10000 0.10000 0.10000
- link LFinger23_link: mass 1e-05 -> 0.00000; geometry collision box size=0.01973 0.01560 0.01069; visual mesh filename=../meshes/stl/LFinger23_0.10.stl scale=0.10000 0.10000 0.10000
- link LForeArm: geometry collision box size=0.07212 0.04968 0.05141; visual mesh filename=../meshes/stl/LElbowRoll_0.10.stl scale=0.10000 0.10000 0.10000
- link LFsrFL_frame: mass 1e-05 -> 0.00000; geometry collision box size=0.01000 0.01000 0.00500; visual box size=0.01000 0.01000 0.00500
- link LFsrFR_frame: mass 1e-05 -> 0.00000; geometry collision box size=0.01000 0.01000 0.00500; visual box size=0.01000 0.01000 0.00500
- link LFsrRL_frame: mass 1e-05 -> 0.00000; geometry collision box size=0.01000 0.01000 0.00500; visual box size=0.01000 0.01000 0.00500
- link LFsrRR_frame: mass 1e-05 -> 0.00000; geometry collision box size=0.01000 0.01000 0.00500; visual box size=0.01000 0.01000 0.00500
- link LHip: geometry collision box size=0.06259 0.03403 0.05367; visual mesh filename=../meshes/stl/LHipRoll_0.10.stl scale=0.10000 0.10000 0.10000
- link LPelvis: geometry collision box size=0.08280 0.05481 0.05852; visual mesh filename=../meshes/stl/LHipYawPitch_0.10.stl scale=0.10000 0.10000 0.10000
- link LShoulder: geometry collision box size=0.06800 0.02418 0.06628; visual mesh filename=../meshes/stl/LShoulderPitch_0.10.stl scale=0.10000 0.10000 0.10000
- link LThigh: geometry collision box size=0.09620 0.09013 0.14907; visual mesh filename=../meshes/stl/LHipPitch_0.10.stl scale=0.10000 0.10000 0.10000
- link LThumb1_link: mass 1e-05 -> 0.00000; geometry collision box size=0.01350 0.01539 0.02155; visual mesh filename=../meshes/stl/LThumb1_0.10.stl scale=0.10000 0.10000 0.10000
- link LThumb2_link: mass 1e-05 -> 0.00000; geometry collision box size=0.01419 0.01579 0.02066; visual mesh filename=../meshes/stl/LThumb2_0.10.stl scale=0.10000 0.10000 0.10000
- link LTibia: geometry collision box size=0.09121 0.09182 0.15120; visual mesh filename=../meshes/stl/LKneePitch_0.10.stl scale=0.10000 0.10000 0.10000
- link Neck: geometry collision box size=0.02520 0.02520 0.02520; visual mesh filename=../meshes/stl/HeadYaw_0.10.stl scale=0.10000 0.10000 0.10000
- link RAnklePitch: geometry collision box size=0.07404 0.03136 0.06433; visual mesh filename=../meshes/stl/RAnklePitch_0.10.stl scale=0.10000 0.10000 0.10000
- link RBicep: geometry collision box size=0.17183 0.06085 0.08297; visual mesh filename=../meshes/stl/RShoulderRoll_0.10.stl scale=0.10000 0.10000 0.10000
- link RFinger11_link: mass 1e-05 -> 0.00000; geometry collision box size=0.01954 0.01567 0.01232; visual mesh filename=../meshes/stl/RFinger11_0.10.stl scale=0.10000 0.10000 0.10000
- link RFinger12_link: mass 1e-05 -> 0.00000; geometry collision box size=0.01954 0.01519 0.01264; visual mesh filename=../meshes/stl/RFinger12_0.10.stl scale=0.10000 0.10000 0.10000
- link RFinger13_link: mass 1e-05 -> 0.00000; geometry collision box size=0.01973 0.01591 0.01120; visual mesh filename=../meshes/stl/RFinger13_0.10.stl scale=0.10000 0.10000 0.10000
- link RFinger21_link: mass 1e-05 -> 0.00000; geometry collision box size=0.01954 0.01599 0.01211; visual mesh filename=../meshes/stl/RFinger21_0.10.stl scale=0.10000 0.10000 0.10000
- link RFinger22_link: mass 1e-05 -> 0.00000; geometry collision box size=0.01954 0.01599 0.01211; visual mesh filename=../meshes/stl/RFinger22_0.10.stl scale=0.10000 0.10000 0.10000
- link RFinger23_link: mass 1e-05 -> 0.00000; geometry collision box size=0.01973 0.01577 0.01118; visual mesh filename=../meshes/stl/RFinger23_0.10.stl scale=0.10000 0.10000 0.10000
- link RForeArm: geometry collision box size=0.07235 0.04878 0.05006; visual mesh filename=../meshes/stl/RElbowRoll_0.10.stl scale=0.10000 0.10000 0.10000
- link RFsrFL_frame: mass 1e-05 -> 0.00000; geometry collision box size=0.01000 0.01000 0.00500; visual box size=0.01000 0.01000 0.00500
- link RFsrFR_frame: mass 1e-05 -> 0.00000; geometry collision box size=0.01000 0.01000 0.00500; visual box size=0.01000 0.01000 0.00500
- link RFsrRL_frame: mass 1e-05 -> 0.00000; geometry collision box size=0.01000 0.01000 0.00500; visual box size=0.01000 0.01000 0.00500
- link RFsrRR_frame: mass 1e-05 -> 0.00000; geometry collision box size=0.01000 0.01000 0.00500; visual box size=0.01000 0.01000 0.00500
- link RHip: geometry collision box size=0.06259 0.03403 0.05367; visual mesh filename=../meshes/stl/RHipRoll_0.10.stl scale=0.10000 0.10000 0.10000
- link RPelvis: geometry collision box size=0.08280 0.05568 0.05907; visual mesh filename=../meshes/stl/RHipYawPitch_0.10.stl scale=0.10000 0.10000 0.10000
- link RShoulder: geometry collision box size=0.06892 0.02440 0.06750; visual mesh filename=../meshes/stl/RShoulderPitch_0.10.stl scale=0.10000 0.10000 0.10000
- link RThigh: geometry collision box size=0.09620 0.09013 0.14906; visual mesh filename=../meshes/stl/RHipPitch_0.10.stl scale=0.10000 0.10000 0.10000
- link RThumb1_link: mass 1e-05 -> 0.00000; geometry collision box size=0.01350 0.01539 0.02155; visual mesh filename=../meshes/stl/RThumb1_0.10.stl scale=0.10000 0.10000 0.10000
- link RThumb2_link: mass 1e-05 -> 0.00000; geometry collision box size=0.01402 0.01579 0.02056; visual mesh filename=../meshes/stl/RThumb2_0.10.stl scale=0.10000 0.10000 0.10000
- link RTibia: geometry collision box size=0.09121 0.09117 0.14870; visual mesh filename=../meshes/stl/RKneePitch_0.10.stl scale=0.10000 0.10000 0.10000
- link l_ankle: geometry collision box size=0.16386 0.09221 0.06587; visual mesh filename=../meshes/stl/LAnkleRoll_0.10.stl scale=0.10000 0.10000 0.10000
- link l_gripper: mass 1e-05 -> 0.00000
- link l_wrist: geometry collision box size=0.08481 0.06829 0.06300; visual mesh filename=../meshes/stl/LWristYaw_0.10.stl scale=0.10000 0.10000 0.10000
- link r_ankle: geometry collision box size=0.16405 0.09226 0.06588; visual mesh filename=../meshes/stl/RAnkleRoll_0.10.stl scale=0.10000 0.10000 0.10000
- link r_gripper: mass 1e-05 -> 0.00000
- link r_wrist: geometry collision box size=0.08469 0.06800 0.06321; visual mesh filename=../meshes/stl/RWristYaw_0.10.stl scale=0.10000 0.10000 0.10000
- link torso: geometry collision box size=0.11168 0.17400 0.23094; visual mesh filename=../meshes/stl/Torso_0.10.stl scale=0.10000 0.10000 0.10000
Joints:
- joint Accelerometer_sensor_fixedjoint: origin xyz=-0.008 0.00606 0.027 rpy=0 0 0 -> xyz=-0.00800 0.00606 0.02700 rpy=0.00000 0.00000 0.00000
- joint CameraBottom_optical_frame_fixedjoint: origin xyz=0 0 0 rpy=-1.5708 0 -1.5708 -> xyz=0.00000 0.00000 0.00000 rpy=-1.57080 -0.00000 -1.57080
- joint CameraBottom_sensor_fixedjoint: origin xyz=0.05071 0 0.01774 rpy=0 0.6929 0 -> xyz=0.05071 0.00000 0.01774 rpy=0.00000 0.69290 0.00000
- joint CameraTop_optical_frame_fixedjoint: origin xyz=0 0 0 rpy=-1.5708 0 -1.5708 -> xyz=-0.00000 0.00000 0.00000 rpy=-1.57080 0.00000 -1.57080
- joint CameraTop_sensor_fixedjoint: origin xyz=0.05871 0 0.06364 rpy=0 0.02094 0 -> xyz=0.05871 0.00000 0.06364 rpy=0.00000 0.02094 0.00000
- joint ChestBoard/Button_sensor_fixedjoint: origin xyz=0.04987 0.00159 0.05516 rpy=0 0 0 -> xyz=0.04987 0.00159 0.05516 rpy=0.00000 0.00000 0.00000
- joint Gyrometer_sensor_fixedjoint: origin xyz=-0.008 0.006 0.029 rpy=0 0 0 -> xyz=-0.00800 0.00600 0.02900 rpy=0.00000 0.00000 0.00000
- joint Head/Touch/Front_sensor_fixedjoint: origin xyz=0.0312 0 0.1014 rpy=0 -1.1861 0 -> xyz=0.03120 0.00000 0.10140 rpy=0.00000 -1.18610 0.00000
- joint Head/Touch/Middle_sensor_fixedjoint: origin xyz=0.001 0 0.1099 rpy=0 -1.5708 0 -> xyz=0.00100 0.00000 0.10990 rpy=3.14159 -1.57079 -3.14159
- joint Head/Touch/Rear_sensor_fixedjoint: origin xyz=-0.0257 0 0.1045 rpy=0 -1.8084 0 -> xyz=-0.02570 0.00000 0.10450 rpy=3.14159 -1.33319 -3.14159
- joint HeadPitch: axis 0 1.0 0 -> 0.00000 1.00000 0.00000; limit lower=-0.67195 upper=0.51487 effort=1.532 velocity=7.19407 -> lower=-0.67195 upper=0.51487 effort=1.53200 velocity=7.19407; origin xyz=0 0 0 rpy=0 0 0 -> xyz=0.00000 0.00000 0.00000 rpy=0.00000 0.00000 0.00000
- joint HeadYaw: axis 0 0 1.0 -> 0.00000 0.00000 1.00000; limit lower=-2.08567 upper=2.08567 effort=1.547 velocity=8.26797 -> lower=-2.08567 upper=2.08567 effort=1.54700 velocity=8.26797; origin xyz=0 0 0.1265 rpy=0 0 0 -> xyz=0.00000 0.00000 0.12650 rpy=0.00000 0.00000 0.00000
- joint InfraredL_sensor_fixedjoint: origin xyz=0.0441 0.0257 0.0466 rpy=0 0 0 -> xyz=0.04410 0.02570 0.04660 rpy=0.00000 0.00000 0.00000
- joint InfraredR_sensor_fixedjoint: origin xyz=0.0441 -0.0257 0.0466 rpy=0 0 0 -> xyz=0.04410 -0.02570 0.04660 rpy=0.00000 0.00000 0.00000
- joint LAnklePitch: axis 0 1.0 0 -> 0.00000 1.00000 0.00000; limit lower=-1.18944 upper=0.92258 effort=3.023 velocity=6.40239 -> lower=-1.18944 upper=0.92258 effort=3.02300 velocity=6.40239; origin xyz=0 0 -0.1029 rpy=0 0 0 -> xyz=0.00000 0.00000 -0.10290 rpy=0.00000 0.00000 0.00000
- joint LAnkleRoll: axis 1.0 0 0 -> 1.00000 0.00000 0.00000; limit lower=-0.39776 upper=0.76899 effort=3.348 velocity=4.16174 -> lower=-0.39776 upper=0.76899 effort=3.34800 velocity=4.16174; origin xyz=0 0 0 rpy=0 0 0 -> xyz=0.00000 0.00000 0.00000 rpy=0.00000 0.00000 0.00000
- joint LElbowRoll: axis 0 0 1.0 -> 0.00000 0.00000 1.00000; limit lower=-1.54462 upper=-0.03491 effort=1.532 velocity=7.19407 -> lower=-1.54462 upper=-0.03491 effort=1.53200 velocity=7.19407; origin xyz=0 0 0 rpy=0 0 0 -> xyz=0.00000 0.00000 0.00000 rpy=0.00000 0.00000 0.00000
- joint LElbowYaw: axis 1.0 0 0 -> 1.00000 0.00000 0.00000; limit lower=-2.08567 upper=2.08567 effort=1.547 velocity=8.26797 -> lower=-2.08567 upper=2.08567 effort=1.54700 velocity=8.26797; origin xyz=0.105 0.015 0 rpy=0 0 0 -> xyz=0.10500 0.01500 0.00000 rpy=0.00000 0.00000 0.00000
- joint LFinger11: axis 0 0 1.0 -> 0.00000 0.00000 1.00000; limit (none) -> lower=0.00000 upper=0.00000 effort=0.00000 velocity=0.00000; origin xyz=0.06907 0.01157 -0.00304 rpy=1.8862 0.97666 0.26407 -> xyz=0.06907 0.01157 -0.00304 rpy=1.88620 0.97666 0.26407
- joint LFinger12: axis 0 0 1.0 -> 0.00000 0.00000 1.00000; limit (none) -> lower=0.00000 upper=0.00000 effort=0.00000 velocity=0.00000; origin xyz=0.01436 0 0 rpy=0 0 -0.9999 -> xyz=0.01436 -0.00000 0.00000 rpy=0.00000 -0.00000 -0.99990
- joint LFinger13: axis 0 0 1.0 -> 0.00000 0.00000 1.00000; limit (none) -> lower=0.00000 upper=0.00000 effort=0.00000 velocity=0.00000; origin xyz=0.01436 0 0 rpy=0 0 -0.9999 -> xyz=0.01436 -0.00000 -0.00000 rpy=-0.00000 -0.00000 -0.99990
- joint LFinger21: axis 0 0 1.0 -> 0.00000 0.00000 1.00000; limit (none) -> lower=0.00000 upper=0.00000 effort=0.00000 velocity=0.00000
- joint LFinger22: axis 0 0 1.0 -> 0.00000 0.00000 1.00000; limit (none) -> lower=0.00000 upper=0.00000 effort=0.00000 velocity=0.00000; origin xyz=0.01436 0 0 rpy=0 0 -0.9999 -> xyz=0.01436 -0.00000 -0.00000 rpy=-0.00000 0.00000 -0.99990
- joint LFinger23: axis 0 0 1.0 -> 0.00000 0.00000 1.00000; limit (none) -> lower=0.00000 upper=0.00000 effort=0.00000 velocity=0.00000; origin xyz=0.01436 0 0 rpy=0 0 -0.9999 -> xyz=0.01436 -0.00000 -0.00000 rpy=0.00000 -0.00000 -0.99990
- joint LFoot/Bumper/Left_sensor_fixedjoint: origin xyz=0.0876 0.019 -0.0353 rpy=0 0 0 -> xyz=0.08760 0.01900 -0.03530 rpy=0.00000 0.00000 0.00000
- joint LFoot/Bumper/Right_sensor_fixedjoint: origin xyz=0.0876 -0.014 -0.0353 rpy=0 0 0 -> xyz=0.08760 -0.01400 -0.03530 rpy=0.00000 0.00000 0.00000
- joint LFoot/FSR/FrontLeft_sensor_fixedjoint: origin xyz=0.07025 0.0299 -0.04511 rpy=0 0 0 -> xyz=0.07025 0.02990 -0.04511 rpy=0.00000 0.00000 0.00000
- joint LFoot/FSR/FrontRight_sensor_fixedjoint: origin xyz=0.07025 -0.0231 -0.04511 rpy=0 0 0 -> xyz=0.07025 -0.02310 -0.04511 rpy=0.00000 0.00000 0.00000
- joint LFoot/FSR/RearLeft_sensor_fixedjoint: origin xyz=-0.03025 0.0299 -0.04511 rpy=0 0 0 -> xyz=-0.03025 0.02990 -0.04511 rpy=0.00000 0.00000 0.00000
- joint LFoot/FSR/RearRight_sensor_fixedjoint: origin xyz=-0.02965 -0.0191 -0.04511 rpy=0 0 0 -> xyz=-0.02965 -0.01910 -0.04511 rpy=0.00000 0.00000 0.00000
- joint LHand: axis 1.0 0 0 -> 1.00000 0.00000 0.00000; limit lower=0 upper=1.0 effort=0.292 velocity=8.33 -> lower=0 upper=1.00000 effort=0.29200 velocity=8.33000; origin xyz=0.05775 0 -0.01231 rpy=0 0 0 -> xyz=0.05775 -0.00000 -0.01231 rpy=0.00000 0.00000 0.00000
- joint LHand/Touch/Back_sensor_fixedjoint: origin xyz=0.038 0 0.025 rpy=0 -1.57079 0 -> xyz=0.03800 0.00000 0.02500 rpy=-0.00042 -1.57079 0.00012
- joint LHand/Touch/Left_sensor_fixedjoint: origin xyz=0.032 0.025 0.003 rpy=0 0 1.5708 -> xyz=0.03200 0.02500 0.00300 rpy=0.00000 0.00000 1.57080
- joint LHand/Touch/Right_sensor_fixedjoint: origin xyz=0.035 -0.025 0.0035 rpy=0 0 -1.5708 -> xyz=0.03500 -0.02500 0.00350 rpy=0.00000 0.00000 -1.57080
- joint LHipPitch: axis 0 1.0 0 -> 0.00000 1.00000 0.00000; limit lower=-1.53589 upper=0.48398 effort=3.023 velocity=6.40239 -> lower=-1.53589 upper=0.48398 effort=3.02300 velocity=6.40239; origin xyz=0 0 0 rpy=0 0 0 -> xyz=0.00000 0.00000 0.00000 rpy=0.00000 0.00000 0.00000
- joint LHipRoll: axis 1.0 0 0 -> 1.00000 0.00000 0.00000; limit lower=-0.37944 upper=0.79046 effort=3.348 velocity=4.16174 -> lower=-0.37944 upper=0.79046 effort=3.34800 velocity=4.16174; origin xyz=0 0 0 rpy=0 0 0 -> xyz=0.00000 0.00000 0.00000 rpy=0.00000 0.00000 0.00000
- joint LHipYawPitch: axis 0 0.70711 -0.70711 -> 0.00000 0.70711 -0.70711; limit lower=-1.14529 upper=0.74072 effort=3.348 velocity=4.16174 -> lower=-1.14529 upper=0.74072 effort=3.34800 velocity=4.16174; origin xyz=0 0.05 -0.085 rpy=0 0 0 -> xyz=0.00000 0.05000 -0.08500 rpy=0.00000 0.00000 0.00000
- joint LKneePitch: axis 0 1.0 0 -> 0.00000 1.00000 0.00000; limit lower=-0.09233 upper=2.11255 effort=3.023 velocity=6.40239 -> lower=-0.09233 upper=2.11255 effort=3.02300 velocity=6.40239; origin xyz=0 0 -0.1 rpy=0 0 0 -> xyz=0.00000 0.00000 -0.10000 rpy=0.00000 0.00000 0.00000
- joint LLeg_effector_fixedjoint: origin xyz=0 0 -0.04511 rpy=0 0 0 -> xyz=0.00000 0.00000 -0.04511 rpy=0.00000 0.00000 0.00000
- joint LShoulderPitch: axis 0 1.0 0 -> 0.00000 1.00000 0.00000; limit lower=-2.08567 upper=2.08567 effort=1.329 velocity=8.26797 -> lower=-2.08567 upper=2.08567 effort=1.32900 velocity=8.26797; origin xyz=0 0.098 0.1 rpy=0 0 0 -> xyz=0.00000 0.09800 0.10000 rpy=0.00000 0.00000 0.00000
- joint LShoulderRoll: axis 0 0 1.0 -> 0.00000 0.00000 1.00000; limit lower=-0.31416 upper=1.32645 effort=1.7835 velocity=7.19407 -> lower=-0.31416 upper=1.32645 effort=1.78350 velocity=7.19407; origin xyz=0 0 0 rpy=0 0 0 -> xyz=0.00000 0.00000 0.00000 rpy=0.00000 0.00000 0.00000
- joint LThumb1: axis 0 0 1.0 -> 0.00000 0.00000 1.00000; limit (none) -> lower=0.00000 upper=0.00000 effort=0.00000 velocity=0.00000; origin xyz=0.04895 0 -0.02638 rpy=-1.5708 0.0473 0 -> xyz=0.04895 0.00000 -0.02638 rpy=-1.57080 0.04730 -0.00000
- joint LThumb2: axis 0 0 1.0 -> 0.00000 0.00000 1.00000; limit (none) -> lower=0.00000 upper=0.00000 effort=0.00000 velocity=0.00000; origin xyz=0.01436 0 0 rpy=0 0 -0.9999 -> xyz=0.01436 -0.00000 -0.00000 rpy=0.00000 -0.00000 -0.99990
- joint LWristYaw: axis 1.0 0 0 -> 1.00000 0.00000 0.00000; limit lower=-1.82387 upper=1.82387 effort=0.4075 velocity=24.6229 -> lower=-1.82387 upper=1.82387 effort=0.40750 velocity=24.62290; origin xyz=0.05595 0 0 rpy=0 0 0 -> xyz=0.05592 -0.00195 0.00000 rpy=0.00000 0.00000 -0.03491
- joint MicroFront_sensor_fixedjoint: origin xyz=0.041 0 0.091 rpy=0 0 0 -> xyz=0.04100 0.00000 0.09100 rpy=0.00000 0.00000 0.00000
- joint MicroLeft_sensor_fixedjoint: origin xyz=-0.0195 0.0606 0.0331 rpy=0 0 0 -> xyz=-0.01950 0.06060 0.03310 rpy=0.00000 0.00000 0.00000
- joint MicroRear_sensor_fixedjoint: origin xyz=-0.0577 0 0.0693 rpy=0 0 0 -> xyz=-0.05770 0.00000 0.06930 rpy=0.00000 0.00000 0.00000
- joint MicroRight_sensor_fixedjoint: origin xyz=-0.0195 -0.0606 0.0331 rpy=0 0 0 -> xyz=-0.01950 -0.06060 0.03310 rpy=0.00000 0.00000 0.00000
- joint RAnklePitch: axis 0 1.0 0 -> 0.00000 1.00000 0.00000; limit lower=-1.1863 upper=0.93201 effort=3.0226 velocity=6.40239 -> lower=-1.18630 upper=0.93201 effort=3.02260 velocity=6.40239; origin xyz=0 0 -0.1029 rpy=0 0 0 -> xyz=0.00000 0.00000 -0.10290 rpy=0.00000 0.00000 0.00000
- joint RAnkleRoll: axis 1.0 0 0 -> 1.00000 0.00000 0.00000; limit lower=-0.76899 upper=0.39776 effort=3.348 velocity=4.16174 -> lower=-0.76899 upper=0.39776 effort=3.34800 velocity=4.16174; origin xyz=0 0 0 rpy=0 0 0 -> xyz=0.00000 0.00000 0.00000 rpy=0.00000 0.00000 0.00000
- joint RElbowRoll: axis 0 0 1.0 -> 0.00000 0.00000 1.00000; limit lower=0.03491 upper=1.54462 effort=1.532 velocity=7.19407 -> lower=0.03491 upper=1.54462 effort=1.53200 velocity=7.19407; origin xyz=0 0 0 rpy=0 0 0 -> xyz=0.00000 0.00000 0.00000 rpy=0.00000 0.00000 0.00000
- joint RElbowYaw: axis 1.0 0 0 -> 1.00000 0.00000 0.00000; limit lower=-2.08567 upper=2.08567 effort=1.547 velocity=8.26797 -> lower=-2.08567 upper=2.08567 effort=1.54700 velocity=8.26797; origin xyz=0.105 -0.015 0 rpy=0 0 0 -> xyz=0.10500 -0.01500 0.00000 rpy=0.00000 0.00000 0.00000
- joint RFinger11: axis 0 0 1.0 -> 0.00000 0.00000 1.00000; limit (none) -> lower=0.00000 upper=0.00000 effort=0.00000 velocity=0.00000; origin xyz=0.06907 0.01157 -0.00304 rpy=1.8862 0.97666 0.26407 -> xyz=0.06907 0.01157 -0.00304 rpy=1.88620 0.97666 0.26407
- joint RFinger12: axis 0 0 1.0 -> 0.00000 0.00000 1.00000; limit (none) -> lower=0.00000 upper=0.00000 effort=0.00000 velocity=0.00000; origin xyz=0.01436 0 0 rpy=0 0 -0.9999 -> xyz=0.01436 0.00000 0.00000 rpy=-0.00000 0.00000 -0.99990
- joint RFinger13: axis 0 0 1.0 -> 0.00000 0.00000 1.00000; limit (none) -> lower=0.00000 upper=0.00000 effort=0.00000 velocity=0.00000; origin xyz=0.01436 0 0 rpy=0 0 -0.9999 -> xyz=0.01436 -0.00000 -0.00000 rpy=0.00000 -0.00000 -0.99990
- joint RFinger21: axis 0 0 1.0 -> 0.00000 0.00000 1.00000; limit (none) -> lower=0.00000 upper=0.00000 effort=0.00000 velocity=0.00000
- joint RFinger22: axis 0 0 1.0 -> 0.00000 0.00000 1.00000; limit (none) -> lower=0.00000 upper=0.00000 effort=0.00000 velocity=0.00000; origin xyz=0.01436 0 0 rpy=0 0 -0.9999 -> xyz=0.01436 -0.00000 0.00000 rpy=0.00000 -0.00000 -0.99990
- joint RFinger23: axis 0 0 1.0 -> 0.00000 0.00000 1.00000; limit (none) -> lower=0.00000 upper=0.00000 effort=0.00000 velocity=0.00000; origin xyz=0.01436 0 0 rpy=0 0 -0.9999 -> xyz=0.01436 0.00000 0.00000 rpy=0.00000 0.00000 -0.99990
- joint RFoot/Bumper/Left_sensor_fixedjoint: origin xyz=0.0876 0.014 -0.0353 rpy=0 0 0 -> xyz=0.08760 0.01400 -0.03530 rpy=0.00000 0.00000 0.00000
- joint RFoot/Bumper/Right_sensor_fixedjoint: origin xyz=0.0876 -0.019 -0.0353 rpy=0 0 0 -> xyz=0.08760 -0.01900 -0.03530 rpy=0.00000 0.00000 0.00000
- joint RFoot/FSR/FrontLeft_sensor_fixedjoint: origin xyz=0.07025 0.0231 -0.04511 rpy=0 0 0 -> xyz=0.07025 0.02310 -0.04511 rpy=0.00000 0.00000 0.00000
- joint RFoot/FSR/FrontRight_sensor_fixedjoint: origin xyz=0.07025 -0.0299 -0.04511 rpy=0 0 0 -> xyz=0.07025 -0.02990 -0.04511 rpy=0.00000 0.00000 0.00000
- joint RFoot/FSR/RearLeft_sensor_fixedjoint: origin xyz=-0.03025 0.0191 -0.04511 rpy=0 0 0 -> xyz=-0.03025 0.01910 -0.04511 rpy=0.00000 0.00000 0.00000
- joint RFoot/FSR/RearRight_sensor_fixedjoint: origin xyz=-0.02965 -0.0299 -0.04511 rpy=0 0 0 -> xyz=-0.02965 -0.02990 -0.04511 rpy=0.00000 0.00000 0.00000
- joint RHand: axis 1.0 0 0 -> 1.00000 0.00000 0.00000; limit lower=0 upper=1.0 effort=0.292 velocity=8.33 -> lower=0 upper=1.00000 effort=0.29200 velocity=8.33000; origin xyz=0.05775 0 -0.01213 rpy=0 0 0 -> xyz=0.05775 0.00000 -0.01213 rpy=0.00000 0.00000 -0.00000
- joint RHand/Touch/Back_sensor_fixedjoint: origin xyz=0.038 0 0.025 rpy=0 -1.57079 0 -> xyz=0.03800 -0.00000 0.02500 rpy=0.00001 -1.57079 0.00096
- joint RHand/Touch/Left_sensor_fixedjoint: origin xyz=0.032 0.025 0.003 rpy=0 0 1.5708 -> xyz=0.03200 0.02500 0.00300 rpy=0.00000 0.00000 1.57080
- joint RHand/Touch/Right_sensor_fixedjoint: origin xyz=0.035 -0.025 0.0035 rpy=0 0 -1.5708 -> xyz=0.03500 -0.02500 0.00350 rpy=0.00000 0.00000 -1.57080
- joint RHipPitch: axis 0 1.0 0 -> 0.00000 1.00000 0.00000; limit lower=-1.53589 upper=0.48398 effort=3.0226 velocity=6.40239 -> lower=-1.53589 upper=0.48398 effort=3.02260 velocity=6.40239; origin xyz=0 0 0 rpy=0 0 0 -> xyz=0.00000 0.00000 0.00000 rpy=0.00000 0.00000 0.00000
- joint RHipRoll: axis 1.0 0 0 -> 1.00000 0.00000 0.00000; limit lower=-0.79046 upper=0.37944 effort=3.348 velocity=4.16174 -> lower=-0.79046 upper=0.37944 effort=3.34800 velocity=4.16174; origin xyz=0 0 0 rpy=0 0 0 -> xyz=0.00000 0.00000 0.00000 rpy=0.00000 0.00000 0.00000
- joint RHipYawPitch: axis 0 0.70711 0.70711 -> 0.00000 0.70711 0.70711; limit lower=-1.14529 upper=0.74072 effort=3.348 velocity=4.16174 -> lower=-1.14529 upper=0.74072 effort=3.34800 velocity=4.16174; origin xyz=0 -0.05 -0.085 rpy=0 0 0 -> xyz=0.00000 -0.05000 -0.08500 rpy=0.00000 0.00000 0.00000
- joint RKneePitch: axis 0 1.0 0 -> 0.00000 1.00000 0.00000; limit lower=-0.09233 upper=2.11255 effort=3.0226 velocity=6.40239 -> lower=-0.09233 upper=2.11255 effort=3.02260 velocity=6.40239; origin xyz=0 0 -0.1 rpy=0 0 0 -> xyz=0.00000 0.00000 -0.10000 rpy=0.00000 0.00000 0.00000
- joint RLeg_effector_fixedjoint: origin xyz=0 0 -0.04511 rpy=0 0 0 -> xyz=0.00000 0.00000 -0.04511 rpy=0.00000 0.00000 0.00000
- joint RShoulderPitch: axis 0 1.0 0 -> 0.00000 1.00000 0.00000; limit lower=-2.08567 upper=2.08567 effort=1.329 velocity=8.26797 -> lower=-2.08567 upper=2.08567 effort=1.32900 velocity=8.26797; origin xyz=0 -0.098 0.1 rpy=0 0 0 -> xyz=0.00000 -0.09800 0.10000 rpy=0.00000 0.00000 0.00000
- joint RShoulderRoll: axis 0 0 1.0 -> 0.00000 0.00000 1.00000; limit lower=-1.32645 upper=0.31416 effort=1.783 velocity=7.19407 -> lower=-1.32645 upper=0.31416 effort=1.78300 velocity=7.19407; origin xyz=0 0 0 rpy=0 0 0 -> xyz=0.00000 0.00000 0.00000 rpy=0.00000 0.00000 0.00000
- joint RThumb1: axis 0 0 1.0 -> 0.00000 0.00000 1.00000; limit (none) -> lower=0.00000 upper=0.00000 effort=0.00000 velocity=0.00000; origin xyz=0.04895 0 -0.02638 rpy=-1.5708 0.0473 0 -> xyz=0.04895 -0.00000 -0.02638 rpy=-1.57080 0.04730 -0.00000
- joint RThumb2: axis 0 0 1.0 -> 0.00000 0.00000 1.00000; limit (none) -> lower=0.00000 upper=0.00000 effort=0.00000 velocity=0.00000; origin xyz=0.01436 0 0 rpy=0 0 -0.9999 -> xyz=0.01436 -0.00000 0.00000 rpy=0.00000 -0.00000 -0.99990
- joint RWristYaw: axis 1.0 0 0 -> 1.00000 0.00000 0.00000; limit lower=-1.82387 upper=1.82387 effort=0.4075 velocity=24.6229 -> lower=-1.82387 upper=1.82387 effort=0.40750 velocity=24.62290; origin xyz=0.05595 0 0 rpy=0 0 0 -> xyz=0.05592 0.00195 0.00000 rpy=0.00000 0.00000 0.03491
- joint base_link_fixedjoint: origin xyz=0 0 0 rpy=0 0 0 -> xyz=0.00000 0.00000 0.00000 rpy=0.00000 0.00000 0.00000
- joint gaze_joint: origin xyz=0.05871 0 0.06364 rpy=0 0 0 -> xyz=0.05871 0.00000 0.06364 rpy=0.00000 0.00000 0.00000
