Commit message: benchmarking

File: data/urdfs/nao/modified/nao.urdf (robot description, URDF)
Before this commit: robot NaoH25V40, 83 links, 82 joints
Links:
- link Head: geometry collision mesh filename=meshes/HeadPitch_0.10.stl scale=0.1 0.1 0.1
- link LAnklePitch: geometry collision mesh filename=meshes/LAnklePitch_0.10.stl scale=0.1 0.1 0.1
- link LBicep: geometry collision mesh filename=meshes/LShoulderRoll_0.10.stl scale=0.1 0.1 0.1
- link LFinger11_link: geometry collision mesh filename=meshes/LFinger11_0.10.stl scale=0.1 0.1 0.1
- link LFinger12_link: geometry collision mesh filename=meshes/LFinger12_0.10.stl scale=0.1 0.1 0.1
- link LFinger13_link: geometry collision mesh filename=meshes/LFinger13_0.10.stl scale=0.1 0.1 0.1
- link LFinger21_link: geometry collision mesh filename=meshes/LFinger21_0.10.stl scale=0.1 0.1 0.1
- link LFinger22_link: geometry collision mesh filename=meshes/LFinger22_0.10.stl scale=0.1 0.1 0.1
- link LFinger23_link: geometry collision mesh filename=meshes/LFinger23_0.10.stl scale=0.1 0.1 0.1
- link LForeArm: geometry collision mesh filename=meshes/LElbowRoll_0.10.stl scale=0.1 0.1 0.1
- link LHip: geometry collision mesh filename=meshes/LHipRoll_0.10.stl scale=0.1 0.1 0.1
- link LPelvis: geometry collision mesh filename=meshes/LHipYawPitch_0.10.stl scale=0.1 0.1 0.1
- link LShoulder: geometry collision mesh filename=meshes/LShoulderPitch_0.10.stl scale=0.1 0.1 0.1
- link LThigh: geometry collision mesh filename=meshes/LHipPitch_0.10.stl scale=0.1 0.1 0.1
- link LThumb1_link: geometry collision mesh filename=meshes/LThumb1_0.10.stl scale=0.1 0.1 0.1
- link LThumb2_link: geometry collision mesh filename=meshes/LThumb2_0.10.stl scale=0.1 0.1 0.1
- link LTibia: geometry collision mesh filename=meshes/LKneePitch_0.10.stl scale=0.1 0.1 0.1
- link Neck: geometry collision mesh filename=meshes/HeadYaw_0.10.stl scale=0.1 0.1 0.1
- link RAnklePitch: geometry collision mesh filename=meshes/RAnklePitch_0.10.stl scale=0.1 0.1 0.1
- link RBicep: geometry collision mesh filename=meshes/RShoulderRoll_0.10.stl scale=0.1 0.1 0.1
- link RFinger11_link: geometry collision mesh filename=meshes/RFinger11_0.10.stl scale=0.1 0.1 0.1
- link RFinger12_link: geometry collision mesh filename=meshes/RFinger12_0.10.stl scale=0.1 0.1 0.1
- link RFinger13_link: geometry collision mesh filename=meshes/RFinger13_0.10.stl scale=0.1 0.1 0.1
- link RFinger21_link: geometry collision mesh filename=meshes/RFinger21_0.10.stl scale=0.1 0.1 0.1
- link RFinger22_link: geometry collision mesh filename=meshes/RFinger22_0.10.stl scale=0.1 0.1 0.1
- link RFinger23_link: geometry collision mesh filename=meshes/RFinger23_0.10.stl scale=0.1 0.1 0.1
- link RForeArm: geometry collision mesh filename=meshes/RElbowRoll_0.10.stl scale=0.1 0.1 0.1
- link RHip: geometry collision mesh filename=meshes/RHipRoll_0.10.stl scale=0.1 0.1 0.1
- link RPelvis: geometry collision mesh filename=meshes/RHipYawPitch_0.10.stl scale=0.1 0.1 0.1
- link RShoulder: geometry collision mesh filename=meshes/RShoulderPitch_0.10.stl scale=0.1 0.1 0.1
- link RThigh: geometry collision mesh filename=meshes/RHipPitch_0.10.stl scale=0.1 0.1 0.1
- link RThumb1_link: geometry collision mesh filename=meshes/RThumb1_0.10.stl scale=0.1 0.1 0.1
- link RThumb2_link: geometry collision mesh filename=meshes/RThumb2_0.10.stl scale=0.1 0.1 0.1
- link RTibia: geometry collision mesh filename=meshes/RKneePitch_0.10.stl scale=0.1 0.1 0.1
- link l_ankle: geometry collision mesh filename=meshes/LAnkleRoll_0.10.stl scale=0.1 0.1 0.1
- link l_wrist: geometry collision mesh filename=meshes/LWristYaw_0.10.stl scale=0.1 0.1 0.1
- link r_ankle: geometry collision mesh filename=meshes/RAnkleRoll_0.10.stl scale=0.1 0.1 0.1
- link r_wrist: geometry collision mesh filename=meshes/RWristYaw_0.10.stl scale=0.1 0.1 0.1
- link torso: geometry collision mesh filename=meshes/Torso_0.10.stl scale=0.1 0.1 0.1

File: data/urdfs/ur/modified/mia_hand_on_ur10.urdf (robot description, URDF)
Before this commit: robot mia_hand_on_ur10, 25 links, 24 joints
Links:
- link arm_base: geometry collision box size=0.2 0.2 1.0
- link flange: geometry 
- link index_sensor: geometry collision cylinder length=0.014262123 radius=0.007128498; collision cylinder length=0.030371133 radius=0.007957385
- link little_fle: geometry collision cylinder length=0.029933602 radius=0.007603541; collision cylinder length=0.030442052 radius=0.007827824
- link middle_sensor: geometry collision cylinder length=0.011829435 radius=0.00683449; collision cylinder length=0.038238756 radius=0.008127632
- link palm: geometry collision box size=0.062414549 0.056382477 0.028578509; collision box size=0.072641067 0.047533765 0.033261035
- link ring_fle: geometry collision cylinder length=0.029933617 radius=0.00760354; collision cylinder length=0.03682825 radius=0.007827824
- link thumb_fle: geometry collision cylinder length=0.055018328 radius=0.011694114; collision cylinder length=0.059818495 radius=0.012714386
- link thumb_opp: geometry 
- link ur10_base_link_inertia: geometry collision mesh filename=./meshes/ur10/collision/base.stl
- link ur10_forearm_link: geometry collision mesh filename=./meshes/ur10/collision/forearm.stl
- link ur10_shoulder_link: geometry collision mesh filename=./meshes/ur10/collision/shoulder.stl
- link ur10_upper_arm_link: geometry collision mesh filename=./meshes/ur10/collision/upperarm.stl
- link ur10_wrist_1_link: geometry collision mesh filename=./meshes/ur10/collision/wrist1.stl
- link ur10_wrist_2_link: geometry collision mesh filename=./meshes/ur10/collision/wrist2.stl
- link ur10_wrist_3_link: geometry collision mesh filename=./meshes/ur10/collision/wrist3.stl

File: data/urdfs/ur/modified/mia_hand_on_ur5.urdf (robot description, URDF)
Before this commit: robot mia_hand_on_ur5, 25 links, 24 joints
Links:
- link flange: geometry visual mesh filename=./meshes/stl/UR_flange.stl scale=0.000999999 0.000999999 0.000999999
- link index_sensor: geometry collision cylinder length=0.014262123 radius=0.007128498; collision cylinder length=0.030371133 radius=0.007957385
- link little_fle: geometry collision cylinder length=0.029933602 radius=0.007603541; collision cylinder length=0.030442052 radius=0.007827824
- link middle_sensor: geometry collision cylinder length=0.011829435 radius=0.00683449; collision cylinder length=0.038238756 radius=0.008127632
- link palm: geometry collision box size=0.062414549 0.056382477 0.028578509; collision box size=0.072641067 0.047533765 0.033261035
- link ring_fle: geometry collision cylinder length=0.029933617 radius=0.00760354; collision cylinder length=0.03682825 radius=0.007827824
- link thumb_fle: geometry collision cylinder length=0.055018328 radius=0.011694114; collision cylinder length=0.059818495 radius=0.012714386
- link thumb_opp: geometry visual mesh filename=./meshes/stl/thumb_metacarpus.stl scale=0.000999987 0.000999987 0.000999987

Commit message: uc1 data

File: data/urdfs/mia_hand_on_ur10.urdf (robot description, URDF)
Before this commit: robot mia_hand_on_ur10, 25 links, 24 joints
Links:
- removed link arm_base
Joints:
- removed joint arm_base_to_arm
- removed joint world_to_robot
- added joint world_to_arm: type fixed, parent world, child ur10_base_link, origin xyz=0.00000 0.00000 1.00000 rpy=0.00000 0.00000 0.00000
